File: house midget/house midget.kicad_sch (KiCad schematic)
At the start: 59 parts, among them J1 Conn_01x02, J10 Conn_01x07, J11 Conn_01x07, J2 Conn_01x02, J3 Conn_01x05, J4 Conn_01x03, J5 Conn_01x03, J6 Conn_01x03, J7 Conn_01x03, J8 Conn_01x03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

Commit message: :building_construction: USBC, PROG. PAGE 2
Parts:
- removed R16: 10K, Resistor_THT:R_Axial_DIN0309_L9.0mm_D3.2mm_P15.24mm_Horizontal, symbol Device:R
- added J12: Conn_01x04, symbol Connector_Generic:Conn_01x04
Connections:
- net +3.3V: now also J12.3 (Pin_3)
- net GND: now also J10.7 (Pin_7), J12.4 (Pin_4)
- net GPIO13: now also J12.1 (Pin_1)
- net IO12: now also J12.2 (Pin_2)
- net NO0: now reaches J4.1 (Pin_1)
- net PCOMI: now reaches J4.2 (Pin_2)
- net NC0: now reaches J4.3 (Pin_3)
- net NO5: now reaches J9.1 (Pin_1)
- net PCOM6: now reaches J9.2 (Pin_2)
- net NC5: now reaches J9.3 (Pin_3)
- net NO4: now reaches J8.1 (Pin_1)
- net PCOM5: now reaches J8.2 (Pin_2)
- net NC4: now reaches J8.3 (Pin_3)
- net NO2: now reaches J6.1 (Pin_1)
- net PCOM3: now reaches J6.2 (Pin_2)
- net NC2: now reaches J6.3 (Pin_3)
- net NO1: now reaches J5.1 (Pin_1)
- net PCOM2: now reaches J5.2 (Pin_2)
- net NC1: now reaches J5.3 (Pin_3)
- net INPUT_D1: now reaches J10.1 (Pin_1)
- net INPUT_D2: now reaches J10.2 (Pin_2)
- net INPUT_D3: now reaches J10.3 (Pin_3)
- net INPUT_D4: now reaches J10.4 (Pin_4)
- net INPUT_D5: now reaches J10.5 (Pin_5)
- net INPUT_D6: now reaches J10.6 (Pin_6)
- net NO3: now reaches J7.1 (Pin_1)
- net PCOM4: now reaches J7.2 (Pin_2)
- net NC3: now reaches J7.3 (Pin_3)
Other:
- added sheet page2 (page2.kicad_sch)
- moved on the sheet: D6, J1, J10, J11, J2, J3, J4, J5, J6, J7, J8, J9

Commit message: :alembic:completed output
Parts:
- added J14, J15: Conn_01x08_Socket, symbol Connector:Conn_01x08_Socket
- added J16: Conn_2Rows-09Pins, symbol Connector_Generic:Conn_2Rows-09Pins
- added R66, R67: 10K, Resistor_SMD:R_0201_0603Metric, symbol Device:R
Connections:
- net +3.3V: now also J15.5 (Pin_5), J16.5 (Pin_5), R66.2, R67.1
- net GND: now also J14.1 (Pin_1), J14.8 (Pin_8), J15.2 (Pin_2), J16.8 (Pin_8)
- net SPI_CLK: now also J14.4 (Pin_4)
- net SPI_CS: now also J14.5 (Pin_5)
- net SPI_DIO0: now also J15.6 (Pin_6)
- net SPI_MISO: now also J14.2 (Pin_2)
- net SPI_MOSI: now also J14.3 (Pin_3)
- net SPI_RST: now also J14.6 (Pin_6)
- new net: J16.6 (Pin_6), R67.2
- new net: J14.7 (Pin_7), R66.1
- no-connect marks 6 -> 11
Other:
- moved on the sheet: C3, C4, C5, R2, R3, R4, R5, U3

Commit message: :egg: completed schematics
Parts:
- added BT1: Battery_Cell, symbol Device:Battery_Cell
- added C24, C25: 10uF/10V, Capacitor_Tantalum_SMD:CP_EIA-2012-12_Kemet-R, symbol Device:C
- added C26, C27: 12.5pF/NC, Capacitor_Tantalum_SMD:CP_EIA-2012-12_Kemet-R, symbol Device:C
- added D17, D18: 1N4148WT, Diode_SMD:D_SOD-523, symbol Diode:1N4148WT
- added J17: Conn_01x04_Socket, symbol Connector:Conn_01x04_Socket
- added Q3, Q4: AO3400A, Package_TO_SOT_SMD:SOT-23, symbol Transistor_FET:AO3400A
- added R68, R69, R70, R71, R72, R73: 427, Resistor_SMD:R_01005_0402Metric_Pad0.57x0.30mm_HandSolder, symbol Device:R
- added U19: DS1307N+, Package_DIP:DIP-8_W7.62mm, symbol Timer_RTC:DS1307N+
- added Y1: Crystal, symbol Device:Crystal
Connections:
- net +3.3V: now also J16.7 (Pin_7), C24.1, C25.1, R69.1, R70.1, R72.1, R73.1; no longer J16.5 (Pin_5)
- net -3.3V: now also D17.2 (A), J17.2 (Pin_2)
- net CE_S: now also J16.6 (Pin_6), R67.2
- net GND: now also BT1.2 (-), C24.2, C25.2, J17.1 (Pin_1), U19.4 (GND)
- net SPI_CLK: now also J16.4 (Pin_4)
- net SPI_CS: now also J16.5 (Pin_5)
- net SPI_MISO: now also J16.2 (Pin_2)
- net SPI_MOSI: now also J16.3 (Pin_3)
- net VCC: now also R68.1, R71.1, U19.8 (VCC)
- net IRQ: now reaches J16.1 (Pin_1)
- new net: BT1.1 (+), D18.2 (A)
- new net: C26.2, U19.1 (X1), Y1.2
- new net: C27.2, U19.2 (X2), Y1.1
- new net: Q4.1 (G), R72.2
- new net: Q3.1 (G), R69.2
- new net: C26.1, C27.1
- new net IIC_SCL: J17.3 (Pin_3), Q3.2 (S), R70.2
- new net IIC_SDA: J17.4 (Pin_4), Q4.2 (S), R73.2
- new net SCL_5V: Q3.3 (D), R68.2, U19.6 (SCL)
- new net SDA5V: Q4.3 (D), R71.2, U19.5 (SDA)
- new net VBAT: D17.1 (K), D18.1 (K), U19.3 (VBAT)
- no-connect marks 11 -> 14
Other:
- note added: "11C"
- note added: "DAC"
- note added: "ESP32"
- note added: "INTERFACE"
- note added: "LDO/POWER SUPPLY"
- note added: "RS485"
- note added: "SPI"
- note added: "TEM.HUMI.1"
- note added: "TEM.HUMI.2"
- moved on the sheet: C1, C10, C2, C3, C4, C5, C8, C9, D1, D2, D6, E2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

Commit message: :tada: fintuning the footprint
Parts:
- added C28: 100nF, Capacitor_Tantalum_SMD:CP_EIA-3216-18_Kemet-A, symbol Device:C
- added C29: 22nF/63V, Capacitor_Tantalum_SMD:CP_EIA-3528-21_Kemet-B, symbol Device:C
- added D19: LED, LED_SMD:LED_Cree-XP, symbol Device:LED
- added J18: Conn_01x04, Module:Flipper_Zero_Angled, symbol Connector_Generic:Conn_01x04
- added R74: 10K, Resistor_SMD:R_0805_2012Metric, symbol Device:R
- added S3: B3U-1000P, B3U-1000P:SW_B3U-1000P, symbol B3U-1000P:B3U-1000P
- added U20: WB3S(0NW9WIP5K33MBOLB), C2830108:WB3S-SMD_OEAKA9ADCKYHKZYS, symbol thuya:WB3S(0NW9WIP5K33MBOLB)
- BT1: footprint (none) -> Battery:BatteryHolder_MPD_BH-18650-PC2
- C1, C10, C2, C3: footprint (none) -> Capacitor_Tantalum_SMD:CP_EIA-3216-18_Kemet-A
- C4: footprint Capacitor_THT:CP_Axial_L18.0mm_D8.0mm_P25.00mm_Horizontal -> Capacitor_Tantalum_SMD:CP_EIA-3528-21_Kemet-B
- C5: footprint Capacitor_THT:CP_Axial_L18.0mm_D8.0mm_P25.00mm_Horizontal -> Capacitor_Tantalum_SMD:CP_EIA-2012-12_Kemet-R
- C6, C8: footprint (none) -> Capacitor_Tantalum_SMD:CP_EIA-2012-12_Kemet-R
- C7, C9: footprint (none) -> Capacitor_SMD:C_1825_4564Metric
- D2: footprint (none) -> LED_SMD:LED_Cree-XP
- J1, J10, J11, J12, J14, J15, J17, J2, J3, J4, J5, J6, J7, J8, J9: footprint (none) -> Module:Flipper_Zero_Angled
- J16: footprint (none) -> Module:Flipper_Zero_Straight
- L1: footprint (none) -> Inductor_SMD:L_Sunlord_MWSA0605S
- R1: footprint (none) -> Resistor_SMD:R_1206_3216Metric
- R11, R13, R17: footprint Resistor_THT:R_Axial_DIN0309_L9.0mm_D3.2mm_P15.24mm_Horizontal -> Resistor_SMD:R_0805_2012Metric
- R14, R15: footprint Resistor_THT:R_Axial_DIN0309_L9.0mm_D3.2mm_P15.24mm_Horizontal -> Resistor_SMD:R_1206_3216Metric
- R2, R3, R4, R5: footprint Resistor_SMD:R_1206_3216Metric -> Resistor_SMD:R_0805_2012Metric
- U5: footprint (none) -> 74HCT14D_653:SOIC127P600X175-14N
- Y1: footprint (none) -> Oscillator:Oscillator_SMD_Fox_FT5H_5.0x3.2mm
Connections:
- net +3.3V: now also J18.1 (Pin_1), R74.2, U20.8 (VCC)
- net -3.3V: now also C28.1, C29.1
- net GND: now also C28.2, C29.2, D19.1 (K), J18.4 (Pin_4), S3.2, U20.9 (GND)
- net GPIO13: now also D19.2 (A)
- net IO12: now also R74.1, S3.1
- net TUYA_RX: now also J18.2 (Pin_2), U20.16 (TXD1)
- new net TUYA_TX: J18.3 (Pin_3), U20.15 (RXD1)
- no-connect marks 14 -> 26
