File: house midget/page2.kicad_sch (KiCad schematic)
At the start: 36 parts, among them J13 USB_C_Receptacle_USB2.0_14P, Q1 SS8050, Q2 SS8050, U7 LM224D, U8 CH340C

Commit message: :alembic:completed output
Parts:
- added C19, C20: 100nF, Capacitor_THT:CP_Radial_D8.0mm_P5.00mm, symbol Device:C
- added C21, C22: 100nF, Capacitor_SMD:C_1206_3216Metric, symbol Device:C
- added C23: C_Polarized_Small_US, symbol Device:C_Polarized_Small_US
- added D11, D12, D13, D14, D15, D16: LED, symbol Device:LED
- added K1, K2, K3, K4, K5, K6: SRD-12VDC-SL-C, SRD-12VDC-SL-C:RELAY_SRD-12VDC-SL-C, symbol SRD-12VDC-SL-C:SRD-12VDC-SL-C
- added P: zx-xh2.54, symbol Connector_Generic:Conn_01x04
- added R38, R39, R40, R41, R42, R43: 2K/1206, Resistor_THT:R_Axial_DIN0614_L14.3mm_D5.7mm_P5.08mm_Vertical, symbol Device:R
- added R44, R45, R46, R47, R48, R49: 100K, Resistor_THT:R_Axial_DIN0614_L14.3mm_D5.7mm_P5.08mm_Vertical, symbol Device:R
- added R50, R51, R52, R53: 10K, Resistor_THT:R_Axial_DIN0614_L14.3mm_D5.7mm_P5.08mm_Vertical, symbol Device:R
- added R54, R55, R56, R57, R58, R59, R60, R61, R62, R63, R64, R65: 4.7K, symbol Device:R
- added RN1, RN2: R_Network04, Resistor_THT:R_Array_SIP5, symbol Device:R_Network04
- added U10, U11, U12, U13, U14, U9: LTV-358T, Package_SO:SO-4_4.4x3.6mm_P2.54mm, symbol Isolator:LTV-358T
- added U15, U16: PCF8574P, Package_DIP:DIP-16_W7.62mm, symbol Interface_Expansion:PCF8574P
- added U17: 74HCT14D_653, 74HCT14D_653:SOIC127P600X175-14N, symbol 74hct14d_653:74HCT14D_653
- added U18: ULN2003A, symbol Transistor_Array:ULN2003A
Connections:
- net +12VIN: now also C22.1, C23.1, D11.2 (A), D12.2 (A), D13.2 (A), D14.2 (A), D15.2 (A), D16.2 (A), R44.2, R45.2, R46.2, R47.2, R48.2, R49.2, U10.1, U11.1, U12.1, U13.1, U14.1, U18.9 (COM), U9.1
- net +3.3V: now also C19.1, C20.1, R50.1, R51.1, R52.1, R53.1, R60.2, R61.2, R62.2, R63.2, R64.2, R65.2, RN1.1 (common), U15.3 (A2), U16.16 (VDD), U16.3 (A2)
- net -3.3V: now also P.1 (Pin_1), RN2.1 (common), U15.16 (VDD)
- net GND: now also C19.2, C20.2, C21.2, C22.2, C23.2, P.2 (Pin_2), U10.3, U11.3, U12.3, U13.3, U14.3, U15.1 (A0), U15.2 (A1), U15.8 (GND), U16.1 (A0), U16.2 (A1), U16.8 (GND), U17.7 (GND), U18.7 (I7), U18.8 (GND), U9.3
- new net: D11.1 (K), R54.1
- new net: D16.1 (K), R59.1
- new net: D14.1 (K), R57.1
- new net: D13.1 (K), R56.1
- new net: R50.2, U15.13 (~{INT})
- new net: D15.1 (K), R58.1
- new net: R51.2, U16.13 (~{INT})
- new net: D12.1 (K), R55.1
- new net +12V: K1.COIL1, K2.COIL1, K3.COIL1, K4.COIL1, K5.COIL1, K6.COIL1
- new net IIC_SCL: P.3 (Pin_3), R53.2, U15.14 (SCL), U16.14 (SCL)
- new net II_SDA: P.4 (Pin_4), R52.2, U15.15 (SDA), U16.15 (SDA)
- new net IN D1: U9.4
- new net IN D2: U10.4
- new net IN D3: U11.4
- new net IN D4: U12.4
- new net IN D5: U13.4
- new net IN D6: U14.4
- new net IN0A: R38.1, U9.2
- new net IN1A: R39.1, U10.2
- new net IN2A: R40.1, U11.2
- new net IN3A: R41.1, U12.2
- new net IN4A: R42.1, U13.2
- new net IN5A: R43.1, U14.2
- new net INA0A: R47.1
- new net INA1A: R46.1
- new net INA2A: R45.1
- new net INA3A: R44.1
- new net INA4A: R49.1
- new net INA5A: R48.1
- new net INPUT D1: R38.2
- new net INPUT D2: R39.2
- new net INPUT D3: R40.2
- new net INPUT D4: R41.2
- new net INPUT D5: R42.2
- new net INPUT D6: R43.2
- new net IN_D1: R65.1, U16.4 (P0)
- new net IN_D2: R64.1, U16.5 (P1)
- new net IN_D3: R63.1, U16.6 (P2)
- new net IN_D4: R62.1, U16.7 (P3)
- new net IN_D5: R61.1, U16.9 (P4)
- new net IN_D6: R60.1, U16.10 (P5)
- new net NC0: K6.NC
- new net NC1: K5.NC
- new net NC2: K4.NC
- new net NC3: K3.NC
- new net NC4: K2.NC
- new net NC5: K1.NC
- new net NO0: K6.NO
- new net NO1: K5.NO
- new net NO2: K4.NO
- new net NO3: K3.NO
- new net NO4: K2.NO
- new net NO5: K1.NO
- new net OT1: RN1.5 (R4), U15.4 (P0), U17.13 (6A)
- new net OT2: RN1.4 (R3), U15.5 (P1), U17.11 (5A)
- new net OT3: RN1.3 (R2), U15.6 (P2), U17.9 (4A)
- new net OT4: RN1.2 (R1), U15.7 (P3), U17.5 (3A)
- new net OT5: RN2.5 (R4), U15.9 (P4), U17.3 (2A)
- new net OT6: RN2.4 (R3), U15.10 (P5), U17.1 (1A)
- new net OUT1: U17.12 (6Y), U18.6 (I6)
- new net OUT2: U17.10 (5Y), U18.5 (I5)
- new net OUT3: U17.8 (4Y), U18.4 (I4)
- new net OUT4: U17.6 (3Y), U18.3 (I3)
- new net OUT5: U17.4 (2Y), U18.2 (I2)
- new net OUT6: U17.2 (1Y), U18.1 (I1)
- new net PCOM1: K6.COM
- new net PCOM2: K5.COM
- new net PCOM3: K4.COM
- new net PCOM4: K3.COM
- new net PCOM5: K2.COM
- new net PCOM6: K1.COM
- new net RLY1: K6.COIL2, R54.2, U18.16 (O1)
- new net RLY2: K5.COIL2, R55.2, U18.15 (O2)
- new net RLY3: K4.COIL2, R56.2, U18.14 (O3)
- new net RLY4: K3.COIL2, R59.2, U18.13 (O4)
- new net RLY5: K2.COIL2, R57.2, U18.12 (O5)
- new net RLY6: K1.COIL2, R58.2, U18.11 (O6)
- new net VCC: C21.1, U17.14 (VCC)
- no-connect marks 8 -> 17
Other:
- moved on the sheet: C17, C18, J13, Q1, Q2, R30, R31, R32, R33, R34, R35, R36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

Commit message: :egg: completed schematics
Other:
- note added: "ADC"
- note added: "OUTPUT"
- note added: "PROG"
- note added: "USBC"
- moved on the sheet: C21, C22, C23, U17, U18

Commit message: :tada: fintuning the footprint
Parts:
- C11, C12, C13, C14: footprint Capacitor_THT:CP_Radial_D8.0mm_P5.00mm -> Capacitor_Tantalum_SMD:CP_EIA-2012-12_Kemet-R
- C15: footprint Capacitor_THT:CP_Radial_D8.0mm_P5.00mm -> Capacitor_SMD:C_1825_4564Metric
- C16, C19, C20: footprint Capacitor_THT:CP_Radial_D8.0mm_P5.00mm -> Capacitor_Tantalum_SMD:CP_EIA-3216-18_Kemet-A
- C17, C18: footprint Capacitor_Tantalum_SMD:CP_EIA-3216-12_Kemet-S -> Capacitor_Tantalum_SMD:CP_EIA-3216-18_Kemet-A
- C21, C22: footprint Capacitor_SMD:C_1206_3216Metric -> Capacitor_Tantalum_SMD:CP_EIA-3216-18_Kemet-A
- C23: footprint (none) -> Capacitor_SMD:C_1825_4564Metric
- D11, D12, D13, D14, D15, D16: footprint (none) -> LED_SMD:LED_Cree-XP
- J13: footprint (none) -> Connector_USB:USB_C_Receptacle_GCT_USB4105-xx-A_16P_TopMnt_Horizontal
- L2: footprint (none) -> Inductor_SMD:L_Sunlord_MWSA0605S
- P1: renamed from P; footprint (none) -> Inductor_SMD:L_Sunlord_MWSA0605S
- R23, R25, R27, R29: footprint Resistor_THT:R_Axial_DIN0614_L14.3mm_D5.7mm_P5.08mm_Vertical -> Resistor_SMD:R_0805_2012Metric
- R30, R31, R34, R35, R36, R37: footprint Capacitor_Tantalum_SMD:CP_EIA-3216-12_Kemet-S_HandSolder -> Resistor_SMD:R_0805_2012Metric
- R32, R33: footprint Capacitor_Tantalum_SMD:CP_EIA-3216-12_Kemet-S_HandSolder -> Resistor_SMD:R_1218_3246Metric
- R38, R39, R40, R41, R42, R43: footprint Resistor_THT:R_Axial_DIN0614_L14.3mm_D5.7mm_P5.08mm_Vertical -> Resistor_SMD:R_1206_3216Metric
- R44, R45, R46, R47, R48, R49: footprint Resistor_THT:R_Axial_DIN0614_L14.3mm_D5.7mm_P5.08mm_Vertical -> Resistor_SMD:R_1218_3246Metric
- R54, R55, R56, R57, R58, R59, R60, R61, R62, R63, R64, R65: footprint (none) -> Resistor_SMD:R_1206_3216Metric
- U18: footprint (none) -> ULN2003ADE4:SOIC127P600X175-16N
