File: house midget/_autosave-house midget.kicad_pcb (KiCad board)
At the start: 2 copper layers, 167 parts, among them J1 Conn_01x02, J10 Conn_01x07, J11 Conn_01x07, J12 Conn_01x04, J13 USB_C_Receptacle_USB2.0_14P, J14 Conn_01x08_Socket, J15 Conn_01x08_Socket, J16 Conn_2Rows-09Pins, J17 Conn_01x04_Socket, J18 Conn_01x04, J2 Conn_01x02, J3 Conn_01x05, J4 Conn_01x03, J5 Conn_01x03, J6 Conn_01x03, J7 Conn_01x03, J8 Conn_01x03, J9 Conn_01x03, P1 zx-xh2.54, Q1 SS8050, Q2 SS8050, Q3 AO3400A, Q4 AO3400A, U1 XL1509-5.0, U10 LTV-358T, U11 LTV-358T, U12 LTV-358T, U13 LTV-358T, U14 LTV-358T, U15 PCF8574P, U16 PCF8574P, U19 DS1307N+, U2 AMS1117-3.3, U3 ESP32-WROOM-32U, U8 CH340C, U9 LTV-358T, Y1 Crystal

Commit message: :beers:pge 1 Done
Parts:
- moved J16 467.8 mm to (488.5, 371.3), turned to 90 degrees
- moved D2 356.5 mm to (504.1, 190.0)
- moved R1 339.2 mm to (513.0, 189.5), turned to 180 degrees
- moved R66 316.0 mm to (58.2, 252.0)
- moved R20 271.0 mm to (334.4, 37.0), turned to 0 degrees
- moved R67 257.6 mm to (495.7, 358.5), turned to 180 degrees
- moved R19 242.9 mm to (310.4, 45.0), turned to 0 degrees
- moved U2 5.50 mm to (441.0, 187.0)
Routing:
- net -3.3V: track 0.00 -> 32.4 mm
- net /TEPP1: track 0.00 -> 22.9 mm
- net /CE_S: track 0.00 -> 6.86 mm
- net Net-(D2-A): track 0.00 -> 6.28 mm
- net Net-(J14-Pin_7): track 0.00 -> 2.36 mm

Commit message: :beers:pge 1 Done
Parts:
- moved L2 628.3 mm to (252.5, 72.5)
- moved R26 627.2 mm to (238.9, 31.5)
- moved R16 627.1 mm to (238.9, 15.0)
- moved C11 624.7 mm to (260.5, 19.9), turned to -90 degrees
- moved C13 624.0 mm to (262.0, 35.6), turned to -90 degrees
- moved C16 613.9 mm to (280.5, 79.1), turned to -90 degrees
- moved C15 601.8 mm to (268.0, 78.7), turned to -90 degrees
- moved R24 588.1 mm to (277.9, 16.1)
- moved J13 587.3 mm to (266.6, 100.6)
- moved C12 586.3 mm to (299.0, 22.6), turned to -90 degrees
- moved R37 582.2 mm to (277.1, 120.0)
- moved R36 581.4 mm to (277.1, 113.0)
- moved R23 578.0 mm to (266.5, 19.9), turned to -90 degrees
- moved C14 577.0 mm to (309.6, 42.0), turned to -90 degrees
- moved R28 576.7 mm to (289.4, 37.0)
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Routing:
- net VCC_12v_1: track 0.00 -> 37.2 mm
- net /TEPP2: track 0.00 -> 25.9 mm
- net /page2/INPUT_AA2: track 0.00 -> 23.4 mm
- net /page2/INPUT_AA3: track 0.00 -> 22.0 mm
- net /page2/INPUT_AA1: track 0.00 -> 20.6 mm
- net /page2/INPUT_AA4: track 0.00 -> 19.8 mm

Commit message: :beers: DONE WITH PROG AND ADC
Parts:
- moved Q2 618.0 mm to (276.6, 141.5)
- moved Q1 618.0 mm to (275.5, 130.5)
- moved R33 617.7 mm to (276.0, 172.0), turned to -90 degrees
- moved C17 617.6 mm to (284.1, 130.5)
- moved C18 612.3 mm to (286.1, 114.5)
- moved R31 612.3 mm to (261.6, 171.0)
- moved R32 607.6 mm to (277.0, 159.5), turned to -90 degrees
- moved R30 600.4 mm to (262.6, 158.0)
- moved R34 597.7 mm to (267.6, 140.5)
- moved R35 595.1 mm to (267.1, 129.5)
Routing:
- net Net-(R31-Pad2): track 0.00 -> 13.7 mm
- net Net-(R30-Pad2): track 0.00 -> 13.5 mm
Changed lines of the file:
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@@
 	(footprint "Resistor_SMD:R_0805_2012Metric"
 		(layer "F.Cu")
-		(at 848.45 2.42)
+		(at 267.0875 129.5)
 		(descr "Resistor SMD 0805 (2012 Metric), square (rectangular) end terminal, IPC-7351 nominal, (Body size source: IPC-SM-782 page 72, https://www.pcb-3d.com/wordpress/wp-content/uploads/ipc-sm-782a_amendment_1_and_2.pdf), generated with kicad-footprint-generator")
 		(tags "resistor")
@@
 	(footprint "Resistor_SMD:R_1218_3246Metric"
 		(layer "F.Cu")
-		(at 861.87 -23.67)
+		(at 276 172.025 -90)
 		(descr "Resistor SMD 1218 (3246 Metric), square (rectangular) end terminal, IPC-7351 nominal, (Body size source: https://www.vishay.com/docs/20035/dcrcwe3.pdf), generated with kicad-footprint-generator")
 		(tags "resistor")
 		(property "Reference" "R33"
-			(at 0 -3.33 0)
+			(at 0 -3.33 90)
 			(layer "F.SilkS")
 			(effects
@@
 		)
 		(property "Value" "100R"
-			(at 0 3.33 0)
+			(at 0 3.33 90)
 			(layer "F.Fab")
 			(effects
@@
 		)
 		(property "Datasheet" ""
-			(at 0 0 0)
+			(at 0 0 90)
 			(layer "F.Fab")
 			(hide yes)
@@
 		)
 		(property "Description" "Resistor"
-			(at 0 0 0)
+			(at 0 0 90)
 			(layer "F.Fab")
 			(hide yes)
@@
 		(attr smd)
 		(fp_line
-			(start -0.777064 -2.41)
-			(end 0.777064 -2.41)
+			(start -0.777064 2.41)
+			(end 0.777064 2.41)
 			(stroke
 				(width 0.12)
@@
 		)
 		(fp_line
-			(start -0.777064 2.41)
-			(end 0.777064 2.41)
+			(start -0.777064 -2.41)
+			(end 0.777064 -2.41)
 			(stroke
 				(width 0.12)
@@
 		)
 		(fp_line
-			(start -2.25 -2.63)
-			(end 2.25 -2.63)
+			(start -2.25 2.63)
+			(end -2.25 -2.63)
 			(stroke
 				(width 0.05)
@@
 		)
 		(fp_line
-			(start -2.25 2.63)
-			(end -2.25 -2.63)
+			(start 2.25 2.63)
+			(end -2.25 2.63)
 			(stroke
 				(width 0.05)
@@
 		)
 		(fp_line
-			(start 2.25 -2.63)
-			(end 2.25 2.63)
+			(start -2.25 -2.63)
+			(end 2.25 -2.63)
 			(stroke
 				(width 0.05)
@@
 		)
 		(fp_line
-			(start 2.25 2.63)
-			(end -2.25 2.63)
+			(start 2.25 -2.63)
+			(end 2.25 2.63)
 			(stroke
 				(width 0.05)
@@
 		)
 		(fp_line
-			(start -1.6 -2.3)
-			(end 1.6 -2.3)
+			(start -1.6 2.3)
+			(end -1.6 -2.3)
 			(stroke
 				(width 0.1)
@@
 		)
 		(fp_line
-			(start -1.6 2.3)
-			(end -1.6 -2.3)
+			(start 1.6 2.3)
+			(end -1.6 2.3)
 			(stroke
 				(width 0.1)
@@
 		)
 		(fp_line
-			(start 1.6 -2.3)
-			(end 1.6 2.3)
+			(start -1.6 -2.3)
+			(end 1.6 -2.3)
 			(stroke
 				(width 0.1)
@@
 		)
 		(fp_line
-			(start 1.6 2.3)
-			(end -1.6 2.3)
+			(start 1.6 -2.3)
+			(end 1.6 2.3)
 			(stroke
 				(width 0.1)
@@
 		)
 		(fp_text user "${REFERENCE}"
-			(at 0 0 0)
+			(at 0 0 90)
 			(layer "F.Fab")
 			(effects
@@
 		)
 		(pad "1" smd roundrect
-			(at -1.475 0)
+			(at -1.475 0 270)
 			(size 1.05 4.75)
 			(layers "F.Cu" "F.Mask" "F.Paste")
@@
 		)
 		(pad "2" smd roundrect
-			(at 1.475 0)
+			(at 1.475 0 270)
 			(size 1.05 4.75)
 			(layers "F.Cu" "F.Mask" "F.Paste")
@@
 	(footprint "Resistor_SMD:R_0805_2012Metric"
 		(layer "F.Cu")
-		(at 844.04 8.32)
+		(at 262.5875 158)
 		(descr "Resistor SMD 0805 (2012 Metric), square (rectangular) end terminal, IPC-7351 nominal, (Body size source: IPC-SM-782 page 72, https://www.pcb-3d.com/wordpress/wp-content/uploads/ipc-sm-782a_amendment_1_and_2.pdf), generated with kicad-footprint-generator")
 		(tags "resistor")
@@
 	(footprint "Package_TO_SOT_SMD:SOT-23"
 		(layer "F.Cu")
-		(at 885.26 34.49)
+		(at 276.5625 141.5)
 		(descr "SOT, 3 Pin (JEDEC TO-236 Var AB https://www.jedec.org/document_search?search_api_views_fulltext=TO-236), generated with kicad-footprint-generator ipc_gullwing_generator.py")
 		(tags "SOT TO_SOT_SMD")
@@
 	(footprint "Resistor_SMD:R_0805_2012Metric"
 		(layer "F.Cu")
-		(at 848.45 -3.48)
+		(at 261.5875 171)
 		(descr "Resistor SMD 0805 (2012 Metric), square (rectangular) end terminal, IPC-7351 nominal, (Body size source: IPC-SM-782 page 72, https://www.pcb-3d.com/wordpress/wp-content/uploads/ipc-sm-782a_amendment_1_and_2.pdf), generated with kicad-footprint-generator")
 		(tags "resistor")
@@
 	(footprint "Package_TO_SOT_SMD:SOT-23"
 		(layer "F.Cu")
-		(at 885.26 29.865)
+		(at 275.5 130.5)
 		(descr "SOT, 3 Pin (JEDEC TO-236 Var AB https://www.jedec.org/document_search?search_api_views_fulltext=TO-236), generated with kicad-footprint-generator ipc_gullwing_generator.py")
 		(tags "SOT TO_SOT_SMD")
@@
 	(footprint "Capacitor_Tantalum_SMD:CP_EIA-3216-18_Kemet-A"
 		(layer "F.Cu")
-		(at 890.585 13.69)
+		(at 284.1475 130.5)
 		(descr "Tantalum Capacitor SMD Kemet-A (3216-18 Metric), IPC-7352 nominal, (Body size from: http://www.kemet.com/Lists/ProductCatalog/Attachments/253/KEM_TC101_STD.pdf), generated with kicad-footprint-generator")
 		(tags "capacitor tantalum")
@@
 	(footprint "Resistor_SMD:R_1218_3246Metric"
 		(layer "F.Cu")
-		(at 856.32 -23.67)
+		(at 277 159.525 -90)
 		(descr "Resistor SMD 1218 (3246 Metric), square (rectangular) end terminal, IPC-7351 nominal, (Body size source: https://www.vishay.com/docs/20035/dcrcwe3.pdf), generated with kicad-footprint-generator")
 		(tags "resistor")
 		(property "Reference" "R32"
-			(at 0 -3.33 0)
+			(at 0 -3.33 90)
 			(layer "F.SilkS")
 			(effects
@@
 		)
 		(property "Value" "100R"
-			(at 0 3.33 0)
+			(at 0 3.33 90)
 			(layer "F.Fab")
 			(effects
@@
 		)
 		(property "Datasheet" ""
-			(at 0 0 0)
+			(at 0 0 90)
 			(layer "F.Fab")
 			(hide yes)
@@
 		)
 		(property "Description" "Resistor"
-			(at 0 0 0)
+			(at 0 0 90)
 			(layer "F.Fab")
 			(hide yes)
@@
 		(attr smd)
 		(fp_line
-			(start -0.777064 -2.41)
-			(end 0.777064 -2.41)
+			(start -0.777064 2.41)
+			(end 0.777064 2.41)
 			(stroke
 				(width 0.12)
@@
 		)
 		(fp_line
-			(start -0.777064 2.41)
-			(end 0.777064 2.41)
+			(start -0.777064 -2.41)
+			(end 0.777064 -2.41)
 			(stroke
 				(width 0.12)
@@
 		)
 		(fp_line
-			(start -2.25 -2.63)
-			(end 2.25 -2.63)
+			(start -2.25 2.63)
+			(end -2.25 -2.63)
 			(stroke
 				(width 0.05)
@@
 		)
 		(fp_line
-			(start -2.25 2.63)
-			(end -2.25 -2.63)
+			(start 2.25 2.63)
+			(end -2.25 2.63)
 			(stroke
 				(width 0.05)
@@
 		)
 		(fp_line
-			(start 2.25 -2.63)
-			(end 2.25 2.63)
+			(start -2.25 -2.63)
+			(end 2.25 -2.63)
 			(stroke
 				(width 0.05)
@@
 		)
 		(fp_line
-			(start 2.25 2.63)
-			(end -2.25 2.63)
+			(start 2.25 -2.63)
+			(end 2.25 2.63)
 			(stroke
 				(width 0.05)
@@
 		)
 		(fp_line
-			(start -1.6 -2.3)
-			(end 1.6 -2.3)
+			(start -1.6 2.3)
+			(end -1.6 -2.3)
 			(stroke
 				(width 0.1)
@@
 		)
 		(fp_line
-			(start -1.6 2.3)
-			(end -1.6 -2.3)
+			(start 1.6 2.3)
+			(end -1.6 2.3)
 			(stroke
 				(width 0.1)
@@
 		)
 		(fp_line
-			(start 1.6 -2.3)
-			(end 1.6 2.3)
+			(start -1.6 -2.3)
+			(end 1.6 -2.3)
 			(stroke
 				(width 0.1)
@@
 		)
 		(fp_line
-			(start 1.6 2.3)
-			(end -1.6 2.3)
+			(start 1.6 -2.3)
+			(end 1.6 2.3)
 			(stroke
 				(width 0.1)
@@
 		)
 		(fp_text user "${REFERENCE}"
-			(at 0 0 0)
+			(at 0 0 90)
 			(layer "F.Fab")
 			(effects
@@
 		)
 		(pad "1" smd roundrect
-			(at -1.475 0)
+			(at -1.475 0 270)
 			(size 1.05 4.75)
 			(layers "F.Cu" "F.Mask" "F.Paste")
@@
 		)
 		(pad "2" smd roundrect
-			(at 1.475 0)
+			(at 1.475 0 270)
 			(size 1.05 4.75)
 			(layers "F.Cu" "F.Mask" "F.Paste")
@@
 	(footprint "Capacitor_Tantalum_SMD:CP_EIA-3216-18_Kemet-A"
 		(layer "F.Cu")
-		(at 890.585 16.84)
+		(at 286.1475 114.5)
 		(descr "Tantalum Capacitor SMD Kemet-A (3216-18 Metric), IPC-7352 nominal, (Body size from: http://www.kemet.com/Lists/ProductCatalog/Attachments/253/KEM_TC101_STD.pdf), generated with kicad-footprint-generator")
 		(tags "capacitor tantalum")
@@
 	(footprint "Resistor_SMD:R_0805_2012Metric"
 		(layer "F.Cu")
-		(at 848.45 -0.53)
+		(at 267.5875 140.5)
 		(descr "Resistor SMD 0805 (2012 Metric), square (rectangular) end terminal, IPC-7351 nominal, (Body size source: IPC-SM-782 page 72, https://www.pcb-3d.com/wordpress/wp-content/uploads/ipc-sm-782a_amendment_1_and_2.pdf), generated with kicad-footprint-generator")
 		(tags "resistor")
@@
 		(net 105)
 	)
+	(segment
+		(start 276.95 158)
+		(end 277 158.05)
+		(width 0.2)
+		(layer "F.Cu")
+		(net 122)
+	)
+	(segment
+		(start 263.5 158)
+		(end 276.95 158)
+		(width 0.2)
+		(layer "F.Cu")
+		(net 122)
+	)
+	(segment
+		(start 262.95 170.55)
+		(end 262.5 171)
+		(width 0.2)
+		(layer "F.Cu")
+		(net 123)
+	)
+	(segment
+		(start 276 170.55)
+		(end 262.95 170.55)
+		(width 0.2)
+		(layer "F.Cu")
+		(net 123)
+	)
 	(embedded_fonts no)

Commit message: :construction: output added to editor
Parts:
- moved R43 807.2 mm to (58.5, 127.0), turned to 180 degrees
- moved R42 806.5 mm to (59.0, 122.0), turned to 180 degrees
- moved R41 806.1 mm to (59.0, 116.0), turned to 180 degrees
- moved R40 805.9 mm to (59.0, 111.5), turned to 180 degrees
- moved R39 805.6 mm to (59.0, 106.0), turned to 180 degrees
- moved R38 804.8 mm to (59.5, 100.5), turned to 180 degrees
- moved U16 794.8 mm to (50.9, 21.9)
- moved U15 788.8 mm to (50.2, 67.6)
- moved R50 786.1 mm to (73.6, 75.0), turned to 180 degrees
- moved C19 785.6 mm to (105.6, 53.0), turned to -90 degrees
- moved R53 779.1 mm to (78.1, 27.0), turned to 180 degrees
- moved C20 777.7 mm to (113.5, 53.1), turned to -90 degrees
- moved U10 769.5 mm to (74.2, 104.6)
- moved U11 769.5 mm to (74.2, 109.9)
- moved U12 769.5 mm to (74.2, 115.2)
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Routing:
- net +12VIN: track 0.00 -> 89.6 mm
- net +3.3V: track 14.2 -> 56.5 mm
- net unconnected-(R51-Pad2): track 0.00 -> 26.7 mm
- net /page2/II_SDA: track 0.00 -> 25.8 mm
- net GND: track 28.2 -> 45.6 mm
- net /page2/DPP_N: track 0.00 -> 14.9 mm
- net /page2/IIC_SCL: track 0.00 -> 14.5 mm
- net /page2/DPP_P: track 0.00 -> 12.2 mm
- net /page2/IN5A: track 0.00 -> 11.0 mm
- net unconnected-(R50-Pad2): track 0.00 -> 10.8 mm
- net /page2/IN3A: track 0.00 -> 10.7 mm
- net /page2/IN2A: track 0.00 -> 10.6 mm
- net /page2/IN4A: track 0.00 -> 10.6 mm
- net Net-(D11-K): track 0.00 -> 10.6 mm
- net /page2/IN1A: track 0.00 -> 10.6 mm
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