File: house midget/house midget.kicad_pcb (KiCad board)
At the start: 2 copper layers, 167 parts, among them J1 Conn_01x02, J10 Conn_01x07, J11 Conn_01x07, J12 Conn_01x04, J13 USB_C_Receptacle_USB2.0_14P, J14 Conn_01x08_Socket, J15 Conn_01x08_Socket, J16 Conn_2Rows-09Pins, J17 Conn_01x04_Socket, J18 Conn_01x04, J2 Conn_01x02, J3 Conn_01x05, J4 Conn_01x03, J5 Conn_01x03, J6 Conn_01x03, J7 Conn_01x03, J8 Conn_01x03, J9 Conn_01x03, P1 zx-xh2.54, Q1 SS8050, Q2 SS8050, Q3 AO3400A, Q4 AO3400A, U1 XL1509-5.0, U10 LTV-358T, U11 LTV-358T, U12 LTV-358T, U13 LTV-358T, U14 LTV-358T, U15 PCF8574P, U16 PCF8574P, U19 DS1307N+, U2 AMS1117-3.3, U3 ESP32-WROOM-32U, U8 CH340C, U9 LTV-358T, Y1 Crystal

Commit message: :beers:pge 1 Done
Parts:
- moved J16 467.8 mm to (488.5, 371.3), turned to 90 degrees
- moved BT1 379.1 mm to (363.4, 382.0), turned to 0 degrees
- moved R66 316.0 mm to (58.2, 252.0)
- moved R67 257.6 mm to (495.7, 358.5), turned to 180 degrees
- moved D17 216.9 mm to (394.3, 345.5)
- moved D18 215.2 mm to (387.5, 347.8), turned to -90 degrees
- moved C24 57.9 mm to (340.1, 339.5), turned to 90 degrees
- moved C25 55.7 mm to (334.0, 339.6), turned to 90 degrees
Routing:
- net Net-(BT1-+): track 0.00 -> 61.3 mm
- net +3.3V: track 0.00 -> 14.2 mm
- net GND: track 14.8 -> 28.2 mm
- net VBAT: track 0.00 -> 7.41 mm
- net /CE_S: track 0.00 -> 6.86 mm
- net Net-(J14-Pin_7): track 0.00 -> 2.36 mm

Commit message: :construction: output added to editor
Parts:
- moved D15 678.1 mm to (267.0, 249.0), turned to 180 degrees
- moved D16 668.4 mm to (266.9, 227.5), turned to 180 degrees
- moved D14 667.7 mm to (267.0, 239.0), turned to 180 degrees
- moved D13 661.0 mm to (266.6, 214.0), turned to 180 degrees
- moved D12 651.4 mm to (267.0, 205.5), turned to 180 degrees
- moved D11 649.7 mm to (267.1, 195.5), turned to 180 degrees
- moved R58 635.4 mm to (278.5, 249.0)
- moved R57 633.2 mm to (278.0, 239.0)
- moved L2 628.3 mm to (252.5, 72.5)
- moved R26 627.2 mm to (238.9, 31.5)
- moved R16 627.1 mm to (238.9, 15.0)
- moved R59 626.4 mm to (278.0, 227.5)
- moved C11 624.7 mm to (260.5, 19.9), turned to -90 degrees
- moved R56 624.7 mm to (278.5, 214.0)
- moved C13 624.0 mm to (262.0, 35.6), turned to -90 degrees
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Routing:
- net +12VIN: track 0.00 -> 89.6 mm
- net VCC_12v_1: track 0.00 -> 37.2 mm
- net -3.3V: track 0.00 -> 32.3 mm
- net /TEPP2: track 0.00 -> 25.9 mm
- net /page2/INPUT_AA2: track 0.00 -> 23.4 mm
- net /TEPP1: track 0.00 -> 22.9 mm
- net /page2/INPUT_AA3: track 0.00 -> 22.0 mm
- net /page2/INPUT_AA1: track 0.00 -> 20.6 mm
- net /page2/INPUT_AA4: track 0.00 -> 19.8 mm
- net Net-(R31-Pad2): track 0.00 -> 13.7 mm
- net Net-(R30-Pad2): track 0.00 -> 13.5 mm
- net Net-(D11-K): track 0.00 -> 10.6 mm
- net Net-(D12-K): track 0.00 -> 9.88 mm
- net Net-(D13-K): track 0.00 -> 9.07 mm
- net Net-(D15-K): track 0.00 -> 8.68 mm
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
Commit message: :egg: started connecting ic
Parts:
- moved RN1 850.7 mm to (35.0, 72.2), turned to 90 degrees
- moved R62 839.6 mm to (30.0, 45.5), turned to 180 degrees
- moved R64 839.6 mm to (29.0, 34.5), turned to 180 degrees
- moved R65 839.2 mm to (29.0, 30.0), turned to 180 degrees
- moved R63 839.1 mm to (30.0, 40.0), turned to 180 degrees
- moved R60 822.5 mm to (40.5, 45.5), turned to 180 degrees
- moved RN2 818.6 mm to (66.0, 62.0), turned to -90 degrees
- moved R61 813.8 mm to (49.0, 45.5), turned to 180 degrees
- moved R43 807.2 mm to (58.5, 127.0), turned to 180 degrees
- moved R42 806.5 mm to (59.0, 122.0), turned to 180 degrees
- moved R41 806.1 mm to (59.0, 116.0), turned to 180 degrees
- moved R40 805.9 mm to (59.0, 111.5), turned to 180 degrees
- moved R39 805.6 mm to (59.0, 106.0), turned to 180 degrees
- moved R38 804.8 mm to (59.5, 100.5), turned to 180 degrees
- moved U16 794.8 mm to (50.9, 21.9)
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Routing:
- net +3.3V: track 14.2 -> 149.0 mm
- net +12VIN: track 89.6 -> 187.8 mm
- net /page2/II_SDA: track 0.00 -> 62.4 mm
- net /page2/IIC_SCL: track 0.00 -> 50.2 mm
- net unconnected-(R51-Pad2): track 0.00 -> 26.7 mm
- net /page2/IN_D4: track 0.00 -> 22.9 mm
- net /page2/RTS: track 0.00 -> 22.7 mm
- net /page2/IN_D2: track 0.00 -> 22.3 mm
- net /page2/IN_D3: track 0.00 -> 21.7 mm
- net /page2/IN_D6: track 0.00 -> 20.0 mm
- net /page2/IN_D1: track 0.00 -> 18.9 mm
- net GND: track 28.2 -> 45.6 mm
- net /page2/OT1: track 0.00 -> 16.4 mm
- net /page2/OT4: track 0.00 -> 16.4 mm
- net /page2/OT3: track 0.00 -> 16.4 mm
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